File: kicad/blueberrytau.kicad_sch (KiCad schematic)
At the start: 56 parts, among them IC1 SN74LVC1G07DCK, J1 PMIC_DBG, J10 ANALOG IN, J11 EPS/ACS, J2 TE-2201778-1, J3 JTAG, J4 DEBUG, J5 VBUS, J6 GPIO, J7 USB1, J8 SPI/I2C/UART, J9 RF, Q1 MMBT2907*, U1 OSD3358-512M-ICB, U2 TLVH431ACDBZR

Commit message: Rev. 0
Parts:
- removed C3: 10uF, Capacitor_SMD:C_0805_2012Metric, symbol Device:C
- removed C5: 47uF, Capacitor_SMD:C_0805_2012Metric, symbol Device:C
- removed TP5: OSC, TestPoint:TestPoint_Pad_D1.0mm, symbol Connector:TestPoint
- removed U1: OSD3358-512M-ICB, OSD335X-BGA-400, symbol ProjectSyms:OSD3358-512M-ICB
- added C9: 100n, Capacitor_SMD:C_0402_1005Metric, symbol Device:C
- added U1: OSD3358-512M-BSM, OSD335X-BGA-256, symbol ProjectSyms:OSD3358-512M-BSM
- added X1: DSC1121BI5-024.0000, Oscillator:Oscillator_SMD_Fordahl_DFAS15-4Pin_5.0x3.2mm, symbol Oscillator:DFA-S15
- renumbered C6 to C1, C8 to C2, C7 to C3, C2 to C4, C1 to C6, C4 to C7, R3 to R2, R4 to R3, R5 to R4, R2 to R5, TP7 to TP1, TP12 to TP10, TP10 to TP11, TP9 to TP2, TP6 to TP3, TP8 to TP4, TP1 to TP5, TP2 to TP6, TP3 to TP7, TP4 to TP8, TP11 to TP9
Connections:
- net +5V: now also U1.P9 (VIN_USB), U1.R9 (VIN_USB), U1.T9 (VIN_USB)
- net +5VD: now also U1.K6 (SYS_VOUT), U1.K7 (SYS_VOUT), U1.L6 (SYS_VOUT), U1.L7 (SYS_VOUT), U1.M15 (USB1_VBUS)
- net AIN0: now also J10.2 (Pin_2), U1.A8 (AIN0); no longer J10.6 (Pin_6)
- net AIN1: now also J10.4 (Pin_4), U1.B8 (AIN1); no longer J10.2 (Pin_2)
- net AIN2: now also J10.6 (Pin_6), U1.B6 (AIN2); no longer J10.4 (Pin_4)
- net AIN3: now also U1.C6 (AIN3)
- net AIN7_BRIDGE: now also U1.D6 (PMIC_MUX_OUT), U1.D7 (AIN7)
- net GND: now also C9.2, U1.A9 (AGND_ADC), U1.B9 (VREFN), U1.D8 (DGND), U1.D9 (DGND), U1.E10 (DGND), U1.E11 (DGND), U1.E12 (DGND), U1.E5 (DGND), U1.E6 (DGND), U1.E7 (DGND), U1.E8 (DGND), U1.E9 (DGND), U1.F12 (DGND), U1.F5 (DGND), U1.G12 (DGND), U1.G5 (DGND), U1.H12 (DGND), U1.H13 (DGND), U1.H4 (DGND), U1.H5 (DGND), U1.J12 (DGND), U1.J13 (DGND), U1.J4 (DGND), U1.J5 (DGND), U1.K12 (DGND), U1.K5 (DGND), U1.L12 (DGND), U1.L14 (USB1_ID), U1.L5 (DGND), U1.M10 (DGND), U1.M11 (DGND), U1.M12 (DGND), U1.M5 (DGND), U1.M6 (DGND), U1.M7 (DGND), U1.M8 (DGND), U1.M9 (DGND), U1.N15 (OSC0_GND), U1.N8 (DGND), U1.N9 (DGND), X1.2 (GND); no longer J2.10 (SWB), RN4.5
- net GPIO1_12: now also U1.P6 (GPIO1[12])
- net GPIO1_13: now also U1.R6 (GPIO1[13])
- net GPIO1_14: now also U1.T6 (GPIO1[14])
- net GPIO1_15: now also U1.P7 (GPIO1[15])
- net GPIO1_16: now also U1.T12 (GPIO1[16])
- net GPIO1_17: now also U1.R12 (GPIO1[17])
- net GPIO1_18: now also U1.P12 (GPIO1[18])
- net GPIO1_19: now also U1.T13 (GPIO1[19])
- net GPIO1_20: now also U1.R13 (GPIO1[20])
- net GPIO1_21: now also U1.P13 (GPIO1[21])
- net GPIO1_22: now also U1.T14 (GPIO1[22])
- net GPIO1_23: now also U1.R14 (GPIO1[23])
- net GPIO1_24: now also U1.P14 (GPIO1[24])
- net GPIO1_25: now also U1.T15 (GPIO1[25])
- net GPIO1_26: now also U1.R15 (GPIO1[26])
- net GPIO1_27: now also U1.T16 (GPIO1[27])
- net GPIO1_29: now also U1.P3 (GPIO1[29])
- net GPIO3_19: now also U1.B3 (GPIO3[19])
- net GPIO3_20: now also U1.C3 (GPIO3[20])
- net GPIO3_21: now also U1.C4 (GPIO3[21])
- net I2C0_SCL: now also U1.C10 (I2C0_SCL), U1.D10 (PMIC_SCL)
- net I2C0_SDA: now also U1.C11 (I2C0_SDA), U1.D11 (PMIC_SDA)
- net I2C1_SCL: now also U1.C13 (I2C1_SCL)
- net I2C1_SDA: now also U1.C12 (I2C1_SDA)
- net JTAG_EMU0: now also U1.E2 (EMU0)
- net JTAG_EMU1: now also U1.E3 (EMU1)
- net JTAG_TCK: now also U1.D1 (TCK)
- net JTAG_TDI: now also U1.C1 (TDI)
- net JTAG_TDO: now also U1.C2 (TDO)
- net JTAG_TMS: now also U1.D2 (TMS)
- net MDIO_CLK: now also U1.D13 (MDIO_CLK)
- net MDIO_DATA: now also U1.E13 (MDIO_DATA)
- net MMC0_CLK: now also RN5.1, U1.B15 (MMC0_CLK); no longer RN5.3
- net MMC0_CMD: now also RN5.2, U1.B16 (MMC0_CMD); no longer RN6.2
- net MMC0_DAT0: now also RN6.3, U1.A16 (MMC0_DAT0); no longer RN5.2
- net MMC0_DAT1: now also RN6.4, U1.A15 (MMC0_DAT1); no longer RN6.1
- net MMC0_DAT2: now also RN5.4, U1.C16 (MMC0_DAT2); no longer RN6.4
- net MMC0_DAT3: now also RN5.3, U1.C15 (MMC0_DAT3); no longer RN5.4
- net MMC0_SDCD: now also U1.C14 (MMC0_SDCD); no longer J2.9 (SWA), RN5.1
- net PMIC_EXTINT: now also U1.D4 (EXTINTN), U1.E4 (PMIC_NINT)
- net PMIC_EXT_WKUP: now also U1.L4 (PMIC_NWAKEUP), U1.M4 (EXT_WAKEUP)
- net PMIC_LDO_PGD: now also U1.N4 (PMIC_LDO_PGOOD), U1.N5 (RTC_PWRONRSTN)
- net PMIC_PB: now also U1.T11 (PMIC_PB_IN)
- net PMIC_PWR_EN: now also U1.N10 (PMIC_POWER_EN), U1.N11 (PMIC_PWR_EN)
- net PWM0: now also U1.T4 (PWM2A)
- net PWM1: now also U1.P5 (PWM2B)
- net RMII_CLK: now also U1.J14 (RMII1_REFCLK)
- net RMII_CRS: now also U1.F14 (RMII1_CRS_DV)
- net RMII_RXD0: now also U1.E14 (RMII1_RXD0)
- net RMII_RXD1: now also U1.D16 (RMII1_RXD1)
- net RMII_RXER: now also U1.E15 (RMII1_RXER)
- net RMII_TXD0: now also U1.H15 (RMII1_TXD0)
- net RMII_TXD1: now also U1.H14 (RMII1_TXD1)
- net RMII_TXEN: now also U1.G14 (RMII1_TXEN)
- net SPI0_CS: now also U1.A14 (SPI0_CS0)
- net SPI0_MISO: now also U1.B13 (SPI0_D0)
- net SPI0_MOSI: now also U1.B14 (SPI0_D1)
- net SPI0_SCLK: now also U1.A13 (SPI0_SCLK)
- net SPI1_CS: now also U1.B1 (SPI1_CS0)
- net SPI1_MISO: now also U1.A2 (SPI1_D0)
- net SPI1_MOSI: now also U1.B2 (SPI1_D1)
- net SPI1_SCLK: now also U1.A1 (SPI1_SCLK)
- net SYSBOOT_0: now also U1.G3 (SYSBOOT0)
- net SYSBOOT_1: now also RN1.2, U1.G2 (SYSBOOT1); no longer RN1.3
- net SYSBOOT_10: now also RN3.3, U1.K2 (SYSBOOT10); no longer RN3.1
- net SYSBOOT_11: now also U1.K1 (SYSBOOT11)
- net SYSBOOT_12: now also RN4.2, U1.L3 (SYSBOOT12); no longer RN4.4
- net SYSBOOT_13: now also RN4.4, U1.L2 (SYSBOOT13); no longer RN4.3
- net SYSBOOT_14: now also RN4.3, U1.L1 (SYSBOOT14)
- net SYSBOOT_15: now also RN4.1, U1.M3 (SYSBOOT15)
- net SYSBOOT_2: now also RN1.3, U1.G1 (SYSBOOT2); no longer RN1.2
- net SYSBOOT_3: now also U1.H3 (SYSBOOT3)
- net SYSBOOT_4: now also U1.H2 (SYSBOOT4)
- net SYSBOOT_5: now also U1.H1 (SYSBOOT5)
- net SYSBOOT_6: now also U1.J3 (SYSBOOT6)
- net SYSBOOT_7: now also U1.J2 (SYSBOOT7)
- net SYSBOOT_8: now also U1.J1 (SYSBOOT8)
- net SYSBOOT_9: now also RN3.1, U1.K3 (SYSBOOT9); no longer RN3.3
- net UART0_RX: now also U1.A12 (UART0_RXD)
- net UART0_TX: now also U1.B12 (UART0_TXD)
- net UART1_RX: now also J8.8 (Pin_8), U1.A11 (UART1_RXD); no longer J8.7 (Pin_7)
- net UART1_TX: now also J8.7 (Pin_7), U1.B11 (UART1_TXD); no longer J8.8 (Pin_8)
- net UART2_RX: now also U1.H16 (UART2_RXD)
- net UART2_TX: now also U1.E16 (UART2_TXD)
- net USB0_CE: now also U1.K13 (USB0_CE)
- net USB0_DRVVBUS: now also U1.J15 (USB0_DRVVBUS)
- net USB0_ID: now also U1.K14 (USB0_ID)
- net USB0_N: now also U1.K16 (USB0_DM)
- net USB0_P: now also U1.K15 (USB0_DP)
- net USB0_VBUS: now also U1.J16 (USB0_VBUS)
- net USB1_N: now also U1.L16 (USB1_DM)
- net USB1_P: now also U1.L15 (USB1_DP)
- net VBAT_NC: now also U1.N7 (PMIC_BAT_SENSE), U1.P8 (VIN_BAT), U1.R8 (VIN_BAT), U1.T8 (VIN_BAT)
- net VBUS: now also U1.P10 (VIN_AC), U1.R10 (VIN_AC), U1.T10 (VIN_AC)
- net VDD_1V8: now also U1.A7 (SYS_ADC_1P8V), U1.B7 (VREFP), U1.F10 (SYS_VDD_1P8V), U1.G10 (SYS_VDD_1P8V), U1.H10 (SYS_VDD_1P8V), U1.H11 (SYS_VDD_1P8V), U1.J10 (SYS_VDD_1P8V), U1.J11 (SYS_VDD_1P8V), U1.K10 (SYS_VDD_1P8V), U1.L10 (SYS_VDD_1P8V)
- net VDD_3V3A: now also J2.4 (VDD), RN4.5, RN5.5, RN5.6, RN5.7, RN5.8, RN6.5, RN6.6, RN6.7, RN6.8, TP10.1, U1.F6 (SYS_VDD1_3P3V), U1.F7 (SYS_VDD1_3P3V), U1.G6 (SYS_VDD1_3P3V), U1.G7 (SYS_VDD1_3P3V); no longer D1.2 (A)
- net VDD_3V3AUX: now also D1.2 (A), C9.1, U1.F11 (SYS_VDD2_3P3V), U1.G11 (SYS_VDD2_3P3V), X1.1 (Vctrl), X1.4 (V+); no longer TP10.1
- net VDD_3V3B: now also U1.F8 (SYS_VDD3_3P3V), U1.F9 (VDDSHV4), U1.G8 (SYS_VDD3_3P3V), U1.G9 (VDDSHV5), U1.H7 (SYS_VDD3_3P3V), U1.H8 (SYS_VDD3_3P3V), U1.H9 (VDDSHV6), U1.J7 (SYS_VDD3_3P3V), U1.J8 (SYS_VDD3_3P3V), U1.J9 (VDDSHV1), U1.K8 (SYS_VDD3_3P3V), U1.K9 (VDDSHV2), U1.L8 (SYS_VDD3_3P3V), U1.L9 (VDDSHV3); no longer J2.4 (VDD), RN5.5, RN5.6, RN5.7, RN5.8, RN6.5, RN6.6, RN6.7, RN6.8
- net VDD_RTC: now also U1.K11 (SYS_RTC_1P8V), U1.L11 (SYS_RTC_1P8V)
- net ~{EXTRST}: now also U1.R11 (WARMRSTN)
- net ~{JTAG_TRST}: now also U1.D3 (NTRST)
- net ~{PMIC_RST}: now also U1.M13 (PMIC_NRESET)
- net ~{UART1_CTS}: now also U1.B10 (UART1_CTSN)
- net ~{UART1_RTS}: now also U1.A10 (UART1_RTSN)
- net at EPRM_EN1.2: now also U1.M2 (EEPROM_WP)
- net at TP1.1: now also U1.G13 (VDDS_PLL)
- net at TP3.1: now also U1.G4 (VDD_CORE)
- net at TP2.1: now also U1.F13 (VDD_MPU)
- net at TP4.1: now also U1.F4 (VDDS_DDR)
- net at IC1.2 (A): now also U1.N12 (PMIC_PGOOD), U1.P11 (PWRONRSTN)
- net at R1.1: now also U1.M16 (RTC_KALDO_ENN)
- new net OSC_IN: U1.P16 (OSC0_IN), X1.3 (OUT)
- no-connect marks 130 -> 58
Other:
- note added: "Blueberry Tau OSD3358-SM Rev. 0"
- note added: "Boot Code: 0b0100 0000 0001 1100"
- note removed: "Blueberry Tau Rev. 0"
- note removed: "Boot Code: 0b01 00 00 00 00 00 11100"
- moved on the sheet: C6, D1, EPRM_EN1, IC1, Q1, R1, R2, R3, R4, R5, TP1, TP10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

Commit message: Updated microSD slot shield net from earth to ground
Connections:
- net Earth: no longer J2.11 (GND), J2.12 (GND), J2.13 (GND), J2.14 (GND), J2.15 (GND), J2.16 (GND)
- net GND: now also J2.11 (GND), J2.12 (GND), J2.13 (GND), J2.14 (GND), J2.15 (GND), J2.16 (GND)
Changed lines of the file:
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@@
   (junction (at 354.33 411.48) (diameter 0) (color 0 0 0 0)
   )
+  (junction (at 530.86 454.66) (diameter 0) (color 0 0 0 0)
+  )
   (junction (at 68.58 91.44) (diameter 0) (color 0 0 0 0)
   )
@@
     (stroke (width 0) (type default) (color 0 0 0 0))
   )
-  (wire (pts (xy 528.32 452.12) (xy 535.94 452.12))
-    (stroke (width 0) (type default) (color 0 0 0 0))
-  )
   (wire (pts (xy 601.98 412.75) (xy 613.41 412.75))
     (stroke (width 0) (type default) (color 0 0 0 0))
@@
     (stroke (width 0) (type default) (color 0 0 0 0))
   )
+  (wire (pts (xy 530.86 452.12) (xy 530.86 454.66))
+    (stroke (width 0) (type default) (color 0 0 0 0))
+  )
   (wire (pts (xy 421.64 267.97) (xy 421.64 273.05))
     (stroke (width 0) (type default) (color 0 0 0 0))
@@
     (stroke (width 0) (type default) (color 0 0 0 0))
   )
-  (wire (pts (xy 535.94 452.12) (xy 535.94 458.47))
-    (stroke (width 0) (type default) (color 0 0 0 0))
-  )
   (wire (pts (xy 209.55 483.87) (xy 238.76 483.87))
     (stroke (width 0) (type default) (color 0 0 0 0))
@@
     (stroke (width 0) (type default) (color 0 0 0 0))
   )
+  (wire (pts (xy 528.32 452.12) (xy 530.86 452.12))
+    (stroke (width 0) (type default) (color 0 0 0 0))
+  )
   (wire (pts (xy 198.12 318.77) (xy 205.74 318.77))
     (stroke (width 0) (type default) (color 0 0 0 0))
@@
     (pin "1")
   )
-  (symbol (lib_id "power:Earth") (at 535.94 458.47 0) (unit 1)
-    (in_bom yes) (on_board yes) (fields_autoplaced)
-    (property "Reference" "#PWR019" (id 0) (at 535.94 464.82 0)
-      (effects (font (size 1.27 1.27)) hide)
-    )
-    (property "Value" "Earth" (id 1) (at 535.94 462.28 0)
-      (effects (font (size 1.27 1.27)) hide)
-    )
-    (property "Footprint" "" (id 2) (at 535.94 458.47 0)
-      (effects (font (size 1.27 1.27)) hide)
-    )
-    (property "Datasheet" "~" (id 3) (at 535.94 458.47 0)
-      (effects (font (size 1.27 1.27)) hide)
-    )
-    (pin "1")
-  )
   (symbol (lib_id "Device:C") (at 46.99 85.09 0) (unit 1)
     (in_bom yes) (on_board yes)
@@
       (reference "#PWR018") (unit 1) (value "GND") (footprint "")
     )
-    (path "/be97d3d6-35df-418b-b833-91dc9881328c"
-      (reference "#PWR019") (unit 1) (value "Earth") (footprint "")
-    )
     (path "/752fd2b9-7447-41b7-8239-552b98dfe049"
